Commit message: base_link collision  origin changed
base_link collision origin changed to align it with the visual element

File: ck9_gazebo/urdf/ck9_gazebo.xacro (robot description, xacro)
@@ -60,5 +60,5 @@
     </visual>
     <collision>
-      <origin xyz="0 0 0.034" rpy="0 0 0" />
+      <origin xyz="0.015 0.009 0.034" rpy="0 0 0" />
       <geometry>
         <cylinder radius="${base_radius}" length="${base_len}"/>
